Commit message: GOAL 2: Move model in gazebo via commands

File: src/fleet_description/urdf/arm.xacro (robot description, xacro)
@@ -1,29 +1,13 @@
 <?xml version="1.0"?>
 <robot xmlns:xacro="http://www.ros.org/wiki/xacro">
-    <xacro:macro name="arm_robot" params="prefix">
-        <link name="${prefix}base_link">
-            <visual>
-                <origin xyz="0 0 0.05" />
-                <geometry>
-                    <box size="0.3 0.3 0.1" />
-                </geometry>
-            </visual>
-            <collision>
-                <origin xyz="0 0 0.05" />
-                <geometry>
-                    <box size="0.3 0.3 0.1" />
-                </geometry>
-            </collision>
-            <inertial>
-                <mass value="50" />
-                <inertia ixx="0.5" iyy="0.5" izz="0.5" ixy="0" ixz="0" iyz="0" />
-            </inertial>
-        </link>
+    <xacro:macro name="arm_robot" params="prefix parent_link">
+        <!-- SHOULDER -->
         <joint name="${prefix}shoulder_joint" type="revolute">
-            <parent link="${prefix}base_link" />
+            <parent link="${parent_link}" />
             <child link="${prefix}shoulder_link" />
-            <origin xyz="0 0 0.05" />
+            <origin xyz="-0.1 0 0.15" />
             <axis xyz="0 0 1" />
             <limit lower="-3.14" upper="3.14" effort="300" velocity="1" />
+            <dynamics damping="0.5" friction="0.1" />
         </joint>
         <link name="${prefix}shoulder_link">
@@ -33,4 +17,7 @@
                     <cylinder length="0.4" radius="0.04" />
                 </geometry>
+                <material name="orange">
+                    <color rgba="1.0 0.5 0.0 1.0" />
+                </material>
             </visual>
             <collision>
@@ -41,8 +28,13 @@
             </collision>
             <inertial>
-                <mass value="2" />
-                <inertia ixx="0.02" iyy="0.02" izz="0.02" ixy="0" ixz="0" iyz="0" />
-            </inertial>
-        </link>
+                <mass value="1.2" />
+                <inertia ixx="0.03" iyy="0.03" izz="0.005"
+                    ixy="0" ixz="0" iyz="0" />
+            </inertial>
+            <gazebo>
+                <selfCollide>false</selfCollide>
+            </gazebo>
+        </link>
+        <!-- ELBOW -->
         <joint name="${prefix}elbow_joint" type="revolute">
             <parent link="${prefix}shoulder_link" />
@@ -51,4 +43,5 @@
             <axis xyz="1 0 0" />
             <limit lower="-1.57" upper="1.57" effort="300" velocity="1" />
+            <dynamics damping="0.5" friction="0.1" />
         </joint>
         <link name="${prefix}elbow_link">
@@ -58,4 +51,7 @@
                     <cylinder length="0.4" radius="0.035" />
                 </geometry>
+                <material name="green">
+                    <color rgba="0.0 0.8 0.0 1.0" />
+                </material>
             </visual>
             <collision>
@@ -66,8 +62,13 @@
             </collision>
             <inertial>
-                <mass value="1.5" />
-                <inertia ixx="0.015" iyy="0.015" izz="0.015" ixy="0" ixz="0" iyz="0" />
-            </inertial>
-        </link>
+                <mass value="0.9" />
+                <inertia ixx="0.02" iyy="0.02" izz="0.004"
+                    ixy="0" ixz="0" iyz="0" />
+            </inertial>
+            <gazebo>
+                <selfCollide>false</selfCollide>
+            </gazebo>
+        </link>
+        <!-- FOREARM -->
         <joint name="${prefix}forearm_joint" type="revolute">
             <parent link="${prefix}elbow_link" />
@@ -76,4 +77,5 @@
             <axis xyz="1 0 0" />
             <limit lower="-1.57" upper="1.57" effort="300" velocity="1" />
+            <dynamics damping="0.5" friction="0.1" />
         </joint>
         <link name="${prefix}forearm_link">
@@ -83,4 +85,7 @@
                     <cylinder length="0.3" radius="0.03" />
                 </geometry>
+                <material name="dark_grey">
+                    <color rgba="0.3 0.3 0.3 1.0" />
+                </material>
             </visual>
             <collision>
@@ -91,8 +96,13 @@
             </collision>
             <inertial>
-                <mass value="1" />
-                <inertia ixx="0.01" iyy="0.01" izz="0.01" ixy="0" ixz="0" iyz="0" />
-            </inertial>
-        </link>
+                <mass value="0.6" />
+                <inertia ixx="0.01" iyy="0.01" izz="0.003"
+                    ixy="0" ixz="0" iyz="0" />
+            </inertial>
+            <gazebo>
+                <selfCollide>false</selfCollide>
+            </gazebo>
+        </link>
+        <!-- WRIST PITCH -->
         <joint name="${prefix}wrist_pitch_joint" type="revolute">
             <parent link="${prefix}forearm_link" />
@@ -101,4 +111,5 @@
             <axis xyz="1 0 0" />
             <limit lower="-1.57" upper="1.57" effort="100" velocity="1" />
+            <dynamics damping="0.3" friction="0.05" />
         </joint>
         <link name="${prefix}wrist_pitch_link">
@@ -108,4 +119,7 @@
                     <cylinder length="0.08" radius="0.025" />
                 </geometry>
+                <material name="cyan">
+                    <color rgba="0.0 0.8 0.8 1.0" />
+                </material>
             </visual>
             <collision>
@@ -116,8 +130,13 @@
             </collision>
             <inertial>
-                <mass value="0.4" />
-                <inertia ixx="0.002" iyy="0.002" izz="0.002" ixy="0" ixz="0" iyz="0" />
-            </inertial>
-        </link>
+                <mass value="0.3" />
+                <inertia ixx="0.003" iyy="0.003" izz="0.001"
+                    ixy="0" ixz="0" iyz="0" />
+            </inertial>
+            <gazebo>
+                <selfCollide>false</selfCollide>
+            </gazebo>
+        </link>
+        <!-- WRIST ROLL -->
         <joint name="${prefix}wrist_roll_joint" type="revolute">
             <parent link="${prefix}wrist_pitch_link" />
@@ -126,4 +145,5 @@
             <axis xyz="0 0 1" />
             <limit lower="-3.14" upper="3.14" effort="50" velocity="2" />
+            <dynamics damping="0.3" friction="0.05" />
         </joint>
         <link name="${prefix}wrist_roll_link">
@@ -133,4 +153,7 @@
                     <cylinder length="0.06" radius="0.022" />
                 </geometry>
+                <material name="grey">
+                    <color rgba="0.6 0.6 0.6 1.0" />
+                </material>
             </visual>
             <collision>
@@ -141,6 +164,112 @@
             </collision>
             <inertial>
-                <mass value="0.3" />
-                <inertia ixx="0.001" iyy="0.001" izz="0.001" ixy="0" ixz="0" iyz="0" />
+                <mass value="0.25" />
+                <inertia ixx="0.002" iyy="0.002" izz="0.001"
+                    ixy="0" ixz="0" iyz="0" />
+            </inertial>
+            <gazebo>
+                <selfCollide>false</selfCollide>
+            </gazebo>
+        </link>
+        <!-- ================= GRIPPER ================= -->
+        <!-- WRIST ROLL to GRIPPER BASE -->
+        <joint name="${prefix}gripper_mount_joint" type="fixed">
+            <parent link="${prefix}wrist_roll_link" />
+            <child link="${prefix}gripper_base" />
+            <origin xyz="0 0 0.06" />
+        </joint>
+        <link name="${prefix}gripper_base">
+            <visual>
+                <origin xyz="0 0 0.05" />
+                <geometry>
+                    <box size="0.08 0.08 0.1" />
+                </geometry>
+                <material name="blue">
+                    <color rgba="0.0 0.0 1.0 1.0" />
+                </material>
+            </visual>
+            <collision>
+                <origin xyz="0 0 0.05" />
+                <geometry>
+                    <box size="0.08 0.08 0.1" />
+                </geometry>
+            </collision>
+            <inertial>
+                <origin xyz="0 0 0.05" />
+                <mass value="0.4" />
+                <inertia ixx="0.002" iyy="0.002" izz="0.002" ixy="0" ixz="0" iyz="0" />
+            </inertial>
+        </link>
+        <!-- GRIPPER CAMERA -->
+        <joint name="${prefix}gripper_camera_joint" type="fixed">
+            <parent link="${prefix}gripper_base" />
+            <child link="${prefix}gripper_camera_link" />
+            <origin xyz="0 0 0.08" rpy="0 -1.57 0" />
+        </joint>
+        <link name="${prefix}gripper_camera_link">
+            <visual>
+                <geometry>
+                    <box size="0.04 0.04 0.04" />
+                </geometry>
+            </visual>
+        </link>
+        <!-- LEFT FINGER -->
+        <joint name="${prefix}left_finger_joint" type="prismatic">
+            <parent link="${prefix}gripper_base" />
+            <child link="${prefix}left_finger" />
+            <origin xyz="0 0.012 0.05" />
+            <axis xyz="0 1 0" />
+            <limit lower="0" upper="0.025" effort="100" velocity="0.2" />
+        </joint>
+        <link name="${prefix}left_finger">
+            <visual>
+                <origin xyz="0 0 0.05" />
+                <geometry>
+                    <box size="0.015 0.015 0.1" />
+                </geometry>
+                <material name="blue">
+                    <color rgba="0.0 0.0 1.0 1.0" />
+                </material>
+            </visual>
+            <collision>
+                <origin xyz="0 0 0.05" />
+                <geometry>
+                    <box size="0.015 0.015 0.1" />
+                </geometry>
+            </collision>
+            <inertial>
+                <origin xyz="0 0 0.05" />
+                <mass value="0.05" />
+                <inertia ixx="0.0002" iyy="0.0002" izz="0.0002" ixy="0" ixz="0" iyz="0" />
+            </inertial>
+        </link>
+        <!-- RIGHT FINGER -->
+        <joint name="${prefix}right_finger_joint" type="prismatic">
+            <parent link="${prefix}gripper_base" />
+            <child link="${prefix}right_finger" />
+            <origin xyz="0 -0.012 0.05" />
+            <axis xyz="0 -1 0" />
+            <limit lower="0" upper="0.025" effort="100" velocity="0.2" />
+        </joint>
+        <link name="${prefix}right_finger">
+            <visual>
+                <origin xyz="0 0 0.05" />
+                <geometry>
+                    <box size="0.015 0.015 0.1" />
+                </geometry>
+                <material name="blue">
+                    <color rgba="0.0 0.0 1.0 1.0" />
+                </material>
+            </visual>
+            <collision>
+                <origin xyz="0 0 0.05" />
+                <geometry>
+                    <box size="0.015 0.015 0.1" />
+                </geometry>
+            </collision>
+            <inertial>
+                <origin xyz="0 0 0.05" />
+                <mass value="0.05" />
+                <inertia ixx="0.0002" iyy="0.0002" izz="0.0002" ixy="0" ixz="0" iyz="0" />
             </inertial>
         </link>

File: src/fleet_description/urdf/car.xacro (robot description, xacro)
@@ -2,4 +2,5 @@
 <robot xmlns:xacro="http://www.ros.org/wiki/xacro">
     <xacro:macro name="car_robot" params="prefix">
+        <!-- BASE -->
         <link name="${prefix}base_link">
             <visual>
@@ -8,4 +9,7 @@
                     <box size="0.3 0.2 0.1" />
                 </geometry>
+                <material name="red">
+                    <color rgba="1 1 0 1" />
+                </material>
             </visual>
             <collision>
@@ -16,108 +20,67 @@
             </collision>
             <inertial>
-                <mass value="5" />
-                <inertia ixx="0.1" iyy="0.1" izz="0.1" ixy="0" ixz="0" iyz="0" />
+                <mass value="30.0" />
+                <inertia
+                    ixx="0.18"
+                    iyy="0.25"
+                    izz="0.30"
+                    ixy="0"
+                    ixz="0"
+                    iyz="0" />
             </inertial>
+            <gazebo>
+                <mu1>2.0</mu1>
+                <mu2>2.0</mu2>
+                <kp>1000000.0</kp>
+                <kd>1.0</kd>
+            </gazebo>
+            <gazebo>
+                <gravity>false</gravity>
+            </gazebo>
         </link>
-        <joint name="${prefix}left_wheel_joint" type="continuous">
-            <parent link="${prefix}base_link" />
-            <child link="${prefix}left_wheel" />
-            <origin xyz="0 0.1 0.05" />
-            <axis xyz="0 1 0" />
-            <limit effort="10" velocity="20" />
-        </joint>
-        <link name="${prefix}left_wheel">
-            <visual>
-                <origin rpy="1.5708 0 0" />
-                <geometry>
-                    <cylinder radius="0.05" length="0.02" />
-                </geometry>
-            </visual>
-            <collision>
-                <origin rpy="1.5708 0 0" />
-                <geometry>
-                    <cylinder radius="0.05" length="0.02" />
-                </geometry>
-            </collision>
-            <inertial>
-                <mass value="0.5" />
-                <inertia ixx="0.001" iyy="0.001" izz="0.001" ixy="0" ixz="0" iyz="0" />
-            </inertial>
-        </link>
-        <joint name="${prefix}right_wheel_joint" type="continuous">
-            <parent link="${prefix}base_link" />
-            <child link="${prefix}right_wheel" />
-            <origin xyz="0 -0.1 0.05" />
-            <axis xyz="0 1 0" />
-            <limit effort="10" velocity="20" />
-        </joint>
-        <link name="${prefix}right_wheel">
-            <visual>
-                <origin rpy="1.5708 0 0" />
-                <geometry>
-                    <cylinder radius="0.05" length="0.02" />
-                </geometry>
-            </visual>
-            <collision>
-                <origin rpy="1.5708 0 0" />
-                <geometry>
-                    <cylinder radius="0.05" length="0.02" />
-                </geometry>
-            </collision>
-            <inertial>
-                <mass value="0.5" />
-                <inertia ixx="0.001" iyy="0.001" izz="0.001" ixy="0" ixz="0" iyz="0" />
-            </inertial>
-        </link>
-        <!-- Front Caster -->
-        <link name="${prefix}caster_wheel_front">
-            <visual>
-                <geometry>
-                    <sphere radius="0.03" />
-                </geometry>
-            </visual>
-            <collision>
-                <geometry>
-                    <sphere radius="0.03" />
-                </geometry>
-            </collision>
-            <inertial>
-                <mass value="0.2" />
-                <inertia ixx="0.0001" iyy="0.0001" izz="0.0001"
-                    ixy="0" ixz="0" iyz="0" />
-            </inertial>
-        </link>
-        <joint name="${prefix}caster_front_joint" type="fixed">
-            <parent link="${prefix}base_link" />
-            <child link="${prefix}caster_wheel_front" />
-            <origin xyz="0.12 0 0.03" rpy="0 0 0" />
-        </joint>
-        <!-- Back Caster -->
-        <link name="${prefix}caster_wheel_back">
-            <visual>
-                <geometry>
-                    <sphere radius="0.03" />
-                </geometry>
-            </visual>
-            <collision>
-                <geometry>
-                    <sphere radius="0.03" />
-                </geometry>
-            </collision>
-            <inertial>
-                <mass value="0.2" />
-                <inertia ixx="0.0001" iyy="0.0001" izz="0.0001"
-                    ixy="0" ixz="0" iyz="0" />
-            </inertial>
-        </link>
-        <joint name="${prefix}caster_back_joint" type="fixed">
-            <parent link="${prefix}base_link" />
-            <child link="${prefix}caster_wheel_back" />
-            <origin xyz="-0.12 0 0.03" rpy="0 0 0" />
-        </joint>
-        <!-- LiDAR -->
+        <!-- ================= WHEEL MACRO ================= -->
+        <xacro:macro name="wheel" params="name x y">
+            <joint name="${prefix}${name}_joint" type="continuous">
+                <parent link="${prefix}base_link" />
+                <child link="${prefix}${name}" />
+                <origin xyz="${x} ${y} 0.05" />
+                <axis xyz="0 1 0" />
+            </joint>
+            <link name="${prefix}${name}">
+                <visual>
+                    <origin rpy="1.5708 0 0" />
+                    <geometry>
+                        <cylinder radius="0.05" length="0.02" />
+                    </geometry>
+                </visual>
+                <collision>
+                    <origin rpy="1.5708 0 0" />
+                    <geometry>
+                        <cylinder radius="0.05" length="0.02" />
+                    </geometry>
+                </collision>
+                <inertial>
+                    <mass value="0.5" />
+                    <inertia ixx="0.001" iyy="0.001" izz="0.001"
+                        ixy="0" ixz="0" iyz="0" />
+                </inertial>
+                <gazebo>
+                    <mu1>2.0</mu1>
+                    <mu2>2.0</mu2>
+                </gazebo>
+            </link>
+        </xacro:macro>
+        <!-- ================= 4 WHEELS ================= -->
+        <!-- Front Left -->
+        <xacro:wheel name="front_left_wheel"  x="0.12"  y="0.10"/>
+        <!-- Front Right -->
+        <xacro:wheel name="front_right_wheel" x="0.12"  y="-0.10"/>
+        <!-- Rear Left -->
+        <xacro:wheel name="rear_left_wheel"   x="-0.12" y="0.10"/>
+        <!-- Rear Right -->
+        <xacro:wheel name="rear_right_wheel"  x="-0.12" y="-0.10"/>
+        <!-- ================= LIDAR ================= -->
         <link name="${prefix}lidar_link">
             <visual>
-                <origin xyz="0 0 0.025" />
                 <geometry>
                     <cylinder radius="0.04" length="0.05" />
@@ -125,5 +88,4 @@
             </visual>
             <collision>
-                <origin xyz="0 0 0.025" />
                 <geometry>
                     <cylinder radius="0.04" length="0.05" />
@@ -139,7 +101,7 @@
             <parent link="${prefix}base_link" />
             <child link="${prefix}lidar_link" />
-            <origin xyz="0 0 0.15" rpy="0 0 0" />
+            <origin xyz="0.0 0 0.15" />
         </joint>
-        <!-- Camera -->
+        <!-- ================= CAMERA ================= -->
         <link name="${prefix}camera_link">
             <visual>
@@ -162,5 +124,5 @@
             <parent link="${prefix}base_link" />
             <child link="${prefix}camera_link" />
-            <origin xyz="0.15 0 0.15" rpy="0 0 0" />
+            <origin xyz="0.15 0 0.15" />
         </joint>
     </xacro:macro>

File: src/fleet_description/urdf/world.xacro (robot description, xacro)
@@ -7,11 +7,74 @@
     <xacro:car_robot prefix="car_" />
     <!-- Spawn arm -->
-    <xacro:arm_robot prefix="arm_" />
-    <!-- FIXED JOINT: Attach arm to car -->
-    <joint name="arm_mount_joint" type="fixed">
-        <parent link="car_base_link" />
-        <child link="arm_base_link" />
-        <!-- Position arm on top of car -->
-        <origin xyz="0 0 0.15" rpy="0 0 0"/>
-    </joint>
+    <xacro:arm_robot prefix="arm_" parent_link="car_base_link" />
+    <!-- ROS2 CONTROL -->
+    <ros2_control name="GazeboSimSystem" type="system">
+        <hardware>
+            <plugin>gz_ros2_control/GazeboSimSystem</plugin>
+        </hardware>
+        <joint name="arm_forearm_joint">
+            <command_interface name="position" />
+            <state_interface name="position" />
+            <state_interface name="velocity" />
+        </joint>
+        <joint name="arm_wrist_pitch_joint">
+            <command_interface name="position" />
+            <state_interface name="position" />
+            <state_interface name="velocity" />
+        </joint>
+        <joint name="arm_wrist_roll_joint">
+            <command_interface name="position" />
+            <state_interface name="position" />
+            <state_interface name="velocity" />
+        </joint>
+        <joint name="arm_shoulder_joint">
+            <command_interface name="position" />
+            <state_interface name="position" />
+            <state_interface name="velocity" />
+        </joint>
+        <joint name="arm_elbow_joint">
+            <command_interface name="position" />
+            <state_interface name="position" />
+            <state_interface name="velocity" />
+        </joint>
+        <joint name="arm_left_finger_joint">
+            <command_interface name="position" />
+            <state_interface name="position" />
+            <state_interface name="velocity" />
+        </joint>
+        <joint name="arm_right_finger_joint">
+            <command_interface name="position" />
+            <state_interface name="position" />
+            <state_interface name="velocity" />
+        </joint>
+        <joint name="car_front_left_wheel_joint">
+            <command_interface name="velocity" />
+            <state_interface name="position" />
+            <state_interface name="velocity" />
+        </joint>
+        <joint name="car_front_right_wheel_joint">
+            <command_interface name="velocity" />
+            <state_interface name="position" />
+            <state_interface name="velocity" />
+        </joint>
+        <joint name="car_rear_left_wheel_joint">
+            <command_interface name="velocity" />
+            <state_interface name="position" />
+            <state_interface name="velocity" />
+        </joint>
+        <joint name="car_rear_right_wheel_joint">
+            <command_interface name="velocity" />
+            <state_interface name="position" />
+            <state_interface name="velocity" />
+        </joint>
+    </ros2_control>
+    <!-- REQUIRED FOR GAZEBO HARMONIC -->
+    <gazebo>
+        <plugin filename="libgz_ros2_control-system.so"
+            name="gz_ros2_control::GazeboSimROS2ControlPlugin">
+            <parameters>
+                /home/madhu/ros2_nexus_fleet_ws/install/fleet_description/share/fleet_description/config/controllers.yaml
+            </parameters>
+        </plugin>
+    </gazebo>
 </robot>
