Commit message: Align wrist_roll

File: src/fleet_description/urdf/nexus_fleet.xacro (robot description, xacro)
@@ -308,5 +308,5 @@
         <origin xyz="0 0.012 0.05" />
         <axis xyz="0 1 0" />
-        <limit lower="0" upper="0.025" effort="100" velocity="0.2" />
+        <limit lower="0" upper="3" effort="300" velocity="0.2" />
     </joint>
     <link name="left_finger">
@@ -334,5 +334,5 @@
         <origin xyz="0 -0.012 0.05" />
         <axis xyz="0 -1 0" />
-        <limit lower="0" upper="0.025" effort="100" velocity="0.2" />
+        <limit lower="0" upper="3" effort="300" velocity="0.2" />
     </joint>
     <link name="right_finger">

Commit message: Render the opencv in dock view

File: src/fleet_description/urdf/nexus_fleet.xacro (robot description, xacro)
@@ -308,5 +308,5 @@
         <origin xyz="0 0.012 0.05" />
         <axis xyz="0 1 0" />
-        <limit lower="0" upper="3" effort="300" velocity="0.2" />
+        <limit lower="0" upper="0.05" effort="300" velocity="0.2" />
     </joint>
     <link name="left_finger">
@@ -334,5 +334,5 @@
         <origin xyz="0 -0.012 0.05" />
         <axis xyz="0 -1 0" />
-        <limit lower="0" upper="3" effort="300" velocity="0.2" />
+        <limit lower="0" upper="0.05" effort="300" velocity="0.2" />
     </joint>
     <link name="right_finger">
